File: hardware/knxRoomUnit/knxRoomSensor_MCU.kicad_sch (KiCad schematic)
At the start: 24 parts, among them J1 esp_prog, J2 JTAG, Q1 S8050, Q2 S8050, SW1 rst, SW2 knx_prog, SW3 ui_up, SW4 ui_dw, SW5 ui_ok, U1 ESP32-WROOM-32

Commit message: Initial hardware commit
Parts:
- removed J2: JTAG, Connector_PinHeader_1.27mm:PinHeader_2x05_P1.27mm_Vertical_SMD, symbol Connector:Conn_ARM_JTAG_SWD_10
- added GN1: OpenKNX_BCU, OpenKNX:NanoBCU_PinHeader_SMD_low_profile, symbol OpenKNX:OpenKNX_BCU
- added J1: KNX, OpenKNX:KNX_Connector, symbol Connector_Generic:Conn_01x02
- added R1: 0, Resistor_SMD:R_0805_2012Metric, symbol Device:R
- D3: renamed from D1; value ui_led -> UI
- J2: renamed from J1; value esp_prog -> PROG
- R10: renamed from R3; footprint Resistor_SMD:R_0402_1005Metric -> Resistor_SMD:R_0603_1608Metric
- R11: renamed from R1; footprint Resistor_SMD:R_0402_1005Metric -> Resistor_SMD:R_0603_1608Metric
- R12: renamed from R4; footprint Resistor_SMD:R_0402_1005Metric -> Resistor_SMD:R_0603_1608Metric
- R13: renamed from R8; footprint Resistor_SMD:R_0402_1005Metric -> Resistor_SMD:R_0603_1608Metric
- R14: renamed from R5; footprint Resistor_SMD:R_0402_1005Metric -> Resistor_SMD:R_0603_1608Metric
- R15: renamed from R6; footprint Resistor_SMD:R_0402_1005Metric -> Resistor_SMD:R_0603_1608Metric
- R16: renamed from R9; footprint Resistor_SMD:R_0402_1005Metric -> Resistor_SMD:R_0603_1608Metric
- R17: renamed from R10; footprint Resistor_SMD:R_0402_1005Metric -> Resistor_SMD:R_0603_1608Metric
- R18: renamed from R7; footprint Resistor_SMD:R_0402_1005Metric -> Resistor_SMD:R_0603_1608Metric
- R9: renamed from R2; footprint Resistor_SMD:R_0402_1005Metric -> Resistor_SMD:R_0603_1608Metric
- SW2: renamed from SW3; value ui_up -> UI_UP; footprint WS-TASV:431151008826 -> (none)
- SW3: renamed from SW2; value knx_prog -> KNX_PROG
- SW4: value ui_dw -> UI_DW; footprint WS-TASV:431151008826 -> (none)
- SW5: value ui_ok -> UI_OK; footprint WS-TASV:431151008826 -> (none)
- renumbered C1 to C12, C2 to C13, C3 to C14, U1 to U2
Connections:
- net +3V3: now also R1.1
- net GND: now also GN1.2 (GND), J1.2 (Pin_2)
- net KNX_RX: now also GN1.4 (Rx)
- net KNX_TX: now also GN1.5 (Tx)
- net JTAG_TCK: no longer names the net of U2.16 (IO13)
- net JTAG_TDI: no longer names the net of U2.14 (IO12)
- net JTAG_TDO renamed KNX_SAVE
- net KNX_SAVE: now also GN1.3 (SAVE)
- net JTAG_TMS: no longer names the net of U2.13 (IO14)
- new net: GN1.1 (KNX+), J1.1 (Pin_1)
- new net +3.3VP: GN1.6 (3V3), R1.2
- no-connect marks 8 -> 12
Other:
- moved on the sheet: C12, C13, C14, D3, J2, Q1, Q2, R10, R11, R12, R13, R14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

Commit message: Hardware Update
Connections:
- net at R13.2, SW2.1: now also SW2.3, U2.7 (IO35)
Changed lines of the file:
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@@
   (junction (at 48.26 127) (diameter 0) (color 0 0 0 0)
   )
+  (junction (at 125.73 113.03) (diameter 0) (color 0 0 0 0)
+  )
   (junction (at 54.61 22.86) (diameter 0) (color 0 0 0 0)
   )
@@
   )
   (junction (at 139.7 110.49) (diameter 0) (color 0 0 0 0)
+  )
+  (junction (at 130.81 113.03) (diameter 0) (color 0 0 0 0)
   )
   (junction (at 127 71.12) (diameter 0) (color 0 0 0 0)
@@
     (stroke (width 0) (type default))
   )
+  (wire (pts (xy 125.73 113.03) (xy 130.81 113.03))
+    (stroke (width 0) (type default))
+  )
